File: KiCad/rev1TypeA/rev1TypeA.kicad_pcb (KiCad board)
At the start: 4 copper layers, 53.9 x 34.9 mm, 16 parts, among them J1 Conn_Coaxial, J2 Conn_01x02, J3 Conn_Coaxial, U2 PMA3-83LN+

Commit message: fixed silkscreen
Other:
- board text added: "FRONT TOWARDS ENEMY"
- board text removed: "FRONT TOWARD ENEMY"
Changed lines of the file:
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@@
 		(capping no)
 		(filling no)
-		(zone_defaults)
 		(pcbplotparams
 			(layerselection 0x00000000_00000000_55555555_5755f5ff)
@@
 		)
 	)
-	(gr_text "FRONT \nTOWARD \nENEMY"
+	(gr_text "FRONT \nTOWARDS ENEMY"
 		(at 134.46 84.98 0)
 		(layer "F.SilkS")
@@
 		(layer "F.Cu")
 	)
+	(segment
+		(start 149.15 89.39)
+		(end 147.4 89.39)
+		(width 0.2)
+		(layer "F.Cu")
+		(net "Net-(J2-Pin_2)")
+	)
+	(segment
+		(start 147.4 89.39)
+		(end 146.86 89.93)
+		(width 0.2)
+		(layer "F.Cu")
+		(net "Net-(J2-Pin_2)")
+	)
+	(segment
+		(start 146.86 89.93)
+		(end 146.86 94.1)
+		(width 0.2)
+		(layer "F.Cu")
+		(net "Net-(J2-Pin_2)")
+	)
+	(segment
+		(start 148.23 96.24)
+		(end 146.87 96.24)
+		(width 0.2)
+		(layer "F.Cu")
+		(net "Net-(J2-Pin_2)")
+	)
+	(segment
+		(start 146.87 96.24)
+		(end 146.86 96.25)
+		(width 0.2)
+		(layer "F.Cu")
+		(net "Net-(J2-Pin_2)")
+	)
+	(segment
+		(start 145.57 96.25)
+		(end 145.56 96.24)
+		(width 0.2)
+		(layer "F.Cu")
+		(net "Net-(J2-Pin_2)")
+	)
+	(segment
+		(start 146.86 94.1)
+		(end 148.23 95.47)
+		(width 0.2)
+		(layer "F.Cu")
+		(net "Net-(J2-Pin_2)")
+	)
+	(segment
+		(start 144.45 96.24)
+		(end 144.445 96.245)
+		(width 0.2)
+		(layer "F.Cu")
+		(net "Net-(J2-Pin_2)")
+	)
+	(segment
+		(start 145.56 96.24)
+		(end 144.45 96.24)
+		(width 0.2)
+		(layer "F.Cu")
+		(net "Net-(J2-Pin_2)")
+	)
+	(segment
+		(start 146.86 96.25)
+		(end 145.57 96.25)
+		(width 0.2)
+		(layer "F.Cu")
+		(net "Net-(J2-Pin_2)")
+	)
+	(segment
+		(start 148.23 95.47)
+		(end 148.23 96.24)
+		(width 0.2)
+		(layer "F.Cu")
+		(net "Net-(J2-Pin_2)")
+	)
 	(via
 		(at 142.48 88.35)
@@
 	)
 	(segment
-		(start 108.58 106.9)
-		(end 108.58 100.733584)
-		(width 0.38)
-		(layer "F.Cu")
-		(net "Net-(FL2-P2)")
-	)
-	(segment
-		(start 109.751573 97.905157)
-		(end 110.540001 97.116729)
-		(width 0.38)
-		(layer "F.Cu")
-		(net "Net-(FL2-P2)")
-	)
-	(arc
-		(start 108.58 100.733584)
-		(mid 108.884482 99.20285)
-		(end 109.751573 97.905157)
-		(width 0.38)
-		(layer "F.Cu")
-		(net "Net-(FL2-P2)")
-	)
-	(segment
-		(start 125.017395 92.715568)
-		(end 128.212297 92.715568)
-		(width 0.38)
-		(layer "F.Cu")
-		(net "Net-(FL1-P1)")
-	)
-	(segment
-		(start 125.011827 92.71)
-		(end 125.017395 92.715568)
-		(width 0.2)
-		(layer "F.Cu")
-		(net "Net-(FL1-P1)")
-	)
-	(segment
-		(start 123.875 92.71)
-		(end 125.011827 92.71)
-		(width 0.65)
-		(layer "F.Cu")
-		(net "Net-(FL1-P1)")
-	)
-	(segment
-		(start 128.212297 92.715568)
-		(end 128.216729 92.72)
-		(width 0.2)
-		(layer "F.Cu")
-		(net "Net-(FL1-P1)")
-	)
-	(segment
 		(start 143.475 96.245)
 		(end 143.475 97.435)
@@
 	)
 	(segment
-		(start 108.63 84.716417)
-		(end 108.63 77.11)
-		(width 0.38)
-		(layer "F.Cu")
-		(net "Net-(FL2-P3)")
-	)
-	(segment
-		(start 110.54 88.283271)
-		(end 109.801573 87.544844)
-		(width 0.38)
-		(layer "F.Cu")
-		(net "Net-(FL2-P3)")
-	)
-	(arc
-		(start 109.801573 87.544844)
-		(mid 108.934482 86.247151)
-		(end 108.63 84.716417)
-		(width 0.38)
-		(layer "F.Cu")
-		(net "Net-(FL2-P3)")
-	)
-	(segment
 		(start 122.899432 92.715568)
 		(end 122.905 92.71)
@@
 	)
 	(segment
-		(start 149.15 89.39)
-		(end 147.4 89.39)
-		(width 0.2)
-		(layer "F.Cu")
-		(net "Net-(J2-Pin_2)")
-	)
-	(segment
-		(start 147.4 89.39)
-		(end 146.86 89.93)
-		(width 0.2)
+		(start 108.58 106.9)
+		(end 108.58 100.733584)
+		(width 0.38)
 		(layer "F.Cu")
-		(net "Net-(J2-Pin_2)")
+		(net "Net-(FL2-P2)")
 	)
 	(segment
-		(start 146.86 89.93)
-		(end 146.86 94.1)
-		(width 0.2)
+		(start 109.751573 97.905157)
+		(end 110.540001 97.116729)
+		(width 0.38)
 		(layer "F.Cu")
-		(net "Net-(J2-Pin_2)")
+		(net "Net-(FL2-P2)")
 	)
-	(segment
-		(start 148.23 96.24)
-		(end 146.87 96.24)
-		(width 0.2)
+	(arc
+		(start 108.58 100.733584)
+		(mid 108.884482 99.20285)
+		(end 109.751573 97.905157)
+		(width 0.38)
 		(layer "F.Cu")
-		(net "Net-(J2-Pin_2)")
+		(net "Net-(FL2-P2)")
 	)
 	(segment
-		(start 146.87 96.24)
-		(end 146.86 96.25)
-		(width 0.2)
+		(start 108.63 84.716417)
+		(end 108.63 77.11)
+		(width 0.38)
 		(layer "F.Cu")
-		(net "Net-(J2-Pin_2)")
+		(net "Net-(FL2-P3)")
 	)
 	(segment
-		(start 145.57 96.25)
-		(end 145.56 96.24)
-		(width 0.2)
+		(start 110.54 88.283271)
+		(end 109.801573 87.544844)
+		(width 0.38)
 		(layer "F.Cu")
-		(net "Net-(J2-Pin_2)")
+		(net "Net-(FL2-P3)")
 	)
-	(segment
-		(start 146.86 94.1)
-		(end 148.23 95.47)
-		(width 0.2)
+	(arc
+		(start 109.801573 87.544844)
+		(mid 108.934482 86.247151)
+		(end 108.63 84.716417)
+		(width 0.38)
 		(layer "F.Cu")
-		(net "Net-(J2-Pin_2)")
+		(net "Net-(FL2-P3)")
 	)
 	(segment
-		(start 144.45 96.24)
-		(end 144.445 96.245)
-		(width 0.2)
+		(start 125.017395 92.715568)
+		(end 128.212297 92.715568)
+		(width 0.38)
 		(layer "F.Cu")
-		(net "Net-(J2-Pin_2)")
+		(net "Net-(FL1-P1)")
 	)
 	(segment
-		(start 145.56 96.24)
-		(end 144.45 96.24)
+		(start 125.011827 92.71)
+		(end 125.017395 92.715568)
 		(width 0.2)
 		(layer "F.Cu")
-		(net "Net-(J2-Pin_2)")
+		(net "Net-(FL1-P1)")
 	)
 	(segment
-		(start 146.86 96.25)
-		(end 145.57 96.25)
-		(width 0.2)
+		(start 123.875 92.71)
+		(end 125.011827 92.71)
+		(width 0.65)
 		(layer "F.Cu")
-		(net "Net-(J2-Pin_2)")
+		(net "Net-(FL1-P1)")
 	)
 	(segment
-		(start 148.23 95.47)
-		(end 148.23 96.24)
+		(start 128.212297 92.715568)
+		(end 128.216729 92.72)
 		(width 0.2)
 		(layer "F.Cu")
-		(net "Net-(J2-Pin_2)")
+		(net "Net-(FL1-P1)")
 	)
 	(zone
